File: hardware/blupoi.sch (KiCad schematic (older format))
At the start: 19 parts, among them P1 MICRO-B-USB, P2 CONN_02X05, U1 NRF52832, X1 32MHz

Commit message: Route APA102 VIN traces
Connections:
- net PM_!CHG: now also U1.18 (P0.15)
- net PM_!GOOD: now also U1.17 (P0.14)
- net PM_EN1: now also U1.15 (P0.12)
- net PM_EN2: now also U1.16 (P0.13)
- net PM_ISET: now also U1.14 (P0.11)
- net PM_SWITCH: now also U1.19 (P0.16)
Changed lines of the file:
@@
 F10 "PM_SWITCH" I R 1400 1600 60
 $EndSheet
-Text Label 1500 1100 0    60   ~ 0
-PM_ISET
 Text GLabel 1500 1100 2    60   Input ~ 0
 PM_ISET
@@
 Wire Wire Line
 	6000 6500 5900 6500
+Text GLabel 6800 2600 2    60   Input ~ 0
+PM_ISET
+Text GLabel 6800 2700 2    60   Input ~ 0
+PM_EN1
+Text GLabel 6800 2800 2    60   Input ~ 0
+PM_EN2
+Text GLabel 6800 2900 2    60   Input ~ 0
+PM_!GOOD
+Text GLabel 6800 3000 2    60   Input ~ 0
+PM_!CHG
+Text GLabel 6800 3100 2    60   Input ~ 0
+PM_SWITCH
+Text Label 7750 3500 0    60   ~ 0
+PM_ISET
+Wire Wire Line
+	6800 3100 6700 3100
+Wire Wire Line
+	6700 3000 6800 3000
+Wire Wire Line
+	6800 2900 6700 2900
+Wire Wire Line
+	6700 2800 6800 2800
+Wire Wire Line
+	6800 2700 6700 2700
+Wire Wire Line
+	6700 2600 6800 2600
 $EndSCHEMATC

Commit message: Removed cp2102 IC
Parts:
- added P3: SERIAL, Pin_Headers:Pin_Header_Straight_1x03, symbol CONN_01X03
- P2: footprint (none) -> Pin_Headers:Pin_Header_Straight_2x05
Connections:
- net GND: now also P3.3 (P3)
- net RX: now also P3.1 (P1)
- net TX: now also P3.2 (P2)
Changed lines of the file:
@@
 $Descr A4 11693 8268
 encoding utf-8
-Sheet 1 7
+Sheet 1 6
 Title ""
 Date ""
@@
 Text Notes 9700 750  0    60   ~ 0
 USB Connector
-$Sheet
-S 550  6800 850  850
-U 57A3E76A
-F0 "cp2102" 60
-F1 "cp2102.sch" 60
-F2 "RX" O R 1400 7100 60
-F3 "TX" I R 1400 7200 60
-F4 "USB_D+" I R 1400 7400 60
-F5 "USB_D-" I R 1400 7500 60
-F6 "V3.3" I R 1400 6900 60
-F7 "VUSB" I R 1400 7000 60
-$EndSheet
-Text GLabel 1500 6900 2    60   Input ~ 0
-V3.3
-Wire Wire Line
-	1500 6900 1400 6900
-Text GLabel 1500 7100 2    60   Input ~ 0
-RX
-Wire Wire Line
-	1500 7100 1400 7100
-Text GLabel 1500 7200 2    60   Input ~ 0
-TX
-Wire Wire Line
-	1500 7200 1400 7200
-Text GLabel 1500 7400 2    60   Input ~ 0
-USB_D+
-Wire Wire Line
-	1500 7400 1400 7400
-Text GLabel 1500 7500 2    60   Input ~ 0
-USB_D-
-Wire Wire Line
-	1500 7500 1400 7500
 Wire Wire Line
 	1400 800  1500 800
@@
 Wire Wire Line
 	10350 1600 10250 1600
-Text GLabel 1500 7000 2    60   Input ~ 0
-VUSB
-Wire Wire Line
-	1500 7000 1400 7000
 Text GLabel 6800 1500 2    60   Input ~ 0
 RX
@@
 F 0 "P2" H 5650 6715 50  0000 C CNN
 F 1 "CONN_02X05" H 5650 6624 50  0000 C CNN
-F 2 "" H 5650 5100 50  0001 C CNN
+F 2 "Pin_Headers:Pin_Header_Straight_2x05" H 5650 5100 50  0001 C CNN
 F 3 "" H 5650 5100 50  0000 C CNN
 	1    5650 6300
@@
 Wire Wire Line
 	6700 2600 6800 2600
+$Comp
+L CONN_01X03 P3
+U 1 1 57E0BFF4
+P 7650 5800
+F 0 "P3" H 7727 5841 50  0000 L CNN
+F 1 "SERIAL" H 7727 5750 50  0000 L CNN
+F 2 "Pin_Headers:Pin_Header_Straight_1x03" H 7650 5800 50  0001 C CNN
+F 3 "" H 7650 5800 50  0000 C CNN
+	1    7650 5800
+	1    0    0    -1
+$EndComp
+Text GLabel 7350 5900 0    60   Input ~ 0
+GND
+Wire Wire Line
+	7350 5900 7450 5900
+Text GLabel 7350 5800 0    60   Input ~ 0
+TX
+Text GLabel 7350 5700 0    60   Input ~ 0
+RX
+Wire Wire Line
+	7350 5700 7450 5700
+Wire Wire Line
+	7450 5800 7350 5800
 $EndSCHEMATC

Commit message: Removed 72 LEDs
Parts:
- L1: footprint Capacitors_SMD:C_0603 -> Resistors_SMD:R_0402
Changed lines of the file:
@@
 LIBS:micro_b_usb
 LIBS:blupoi-cache
-EELAYER 25 0
+EELAYER 26 0
 EELAYER END
 $Descr A4 11693 8268
@@
 F 0 "L1" H 3650 3215 50  0000 C CNN
 F 1 "3.9nH" H 3650 3124 50  0000 C CNN
-F 2 "Capacitors_SMD:C_0603" H 3650 3000 50  0001 C CNN
+F 2 "Resistors_SMD:R_0402" H 3650 3000 50  0001 C CNN
 F 3 "" H 3650 3000 50  0000 C CNN
 F 4 "Value" H 3650 3000 60  0001 C CNN "MFG Name"

Commit message: Switched to fat small design
Parts:
- removed ANT2: ANT_NFC, nfc_antenna:nfc_antenna_60x5mm_1.826uH, symbol ANTENNA
- removed C_tune1, C_tune2: TDB, Capacitors_SMD:C_0603_HandSoldering, symbol C_Small
- removed L1: 3.9nH, Resistors_SMD:R_0402, symbol INDUCTOR_SMALL
- added L1: 3.9nH, Capacitors_SMD:C_0402, symbol L_Small
Connections:
- net at C3.1, U1.30 (ANT): now also L1.2
- net at ANT1.2, C_tune3.1: now also L1.1

Commit message: Added mode button
Parts:
- added R12: 10k, Resistors_SMD:R_0603, symbol R_Small
- added SW_MODE1: SW_SPST, kss241glfs:KSS241GLFS, symbol SW_SPST
Connections:
- net GND: now also R12.2
- net V3.3: now also SW_MODE1.2 (B)
- net at U1.12 (P0.10): now also R12.1, SW_MODE1.1 (A)
Changed lines of the file:
@@
 LIBS:micro_b_usb
 LIBS:sip32408
+LIBS:switches
 LIBS:blupoi-cache
 EELAYER 26 0
@@
 Wire Wire Line
 	4250 3950 4600 3950
+$Comp
+L SW_SPST SW_MODE1
+U 1 1 58AA012E
+P 7900 2500
+F 0 "SW_MODE1" H 7900 2550 50  0000 C CNN
+F 1 "SW_SPST" H 7900 2450 50  0000 C CNN
+F 2 "kss241glfs:KSS241GLFS" H 450 0   50  0001 C CNN
+F 3 "" H 450 0   50  0001 C CNN
+	1    7900 2500
+	1    0    0    -1
+$EndComp
+Wire Wire Line
+	6700 2500 7700 2500
+$Comp
+L R_Small R12
+U 1 1 58AA0946
+P 7550 2700
+F 0 "R12" H 7609 2746 50  0000 L CNN
+F 1 "10k" H 7609 2655 50  0000 L CNN
+F 2 "Resistors_SMD:R_0603" H -250 150 50  0001 C CNN
+F 3 "" H -250 150 50  0001 C CNN
+	1    7550 2700
+	1    0    0    -1
+$EndComp
+Wire Wire Line
+	7550 2500 7550 2600
+Connection ~ 7550 2500
+$Comp
+L GND #PWR010
+U 1 1 58AA0D95
+P 7550 2900
+F 0 "#PWR010" H 7600 2950 50  0001 C CNN
+F 1 "GND" H 7555 2727 50  0000 C CNN
+F 2 "" H 0   0   50  0001 C CNN
+F 3 "" H 0   0   50  0001 C CNN
+	1    7550 2900
+	1    0    0    -1
+$EndComp
+Wire Wire Line
+	7550 2900 7550 2800
+Text GLabel 8200 2400 1    60   Input ~ 0
+V3.3
+Wire Wire Line
+	8200 2400 8200 2500
+Wire Wire Line
+	8200 2500 8100 2500
 $EndSCHEMATC

Commit message: Started routing v0.2...
Connections:
- net ACC_I2C_SCL: now also U1.27 (P0.22); no longer U1.8 (P0.06)
- net ACC_I2C_SDA: now also U1.28 (P0.23); no longer U1.9 (P0.07)
- net APA102_0_MOSI: now also U1.5 (P0.03/AIN1); no longer U1.37 (P0.25)
- net APA102_0_SCK: now also U1.4 (P0.02/AIN0); no longer U1.38 (P0.26)
- net APA102_1_MOSI: now also U1.7 (P0.05/AIN3); no longer U1.39 (P0.27)
- net APA102_1_SCK: now also U1.6 (P0.04/AIN2); no longer U1.40 (P0.28/AIN4)
- net MIC_I2S_SCK: now also U1.9 (P0.07); no longer U1.27 (P0.22)
- net MIC_I2S_SD: now also U1.10 (P0.08); no longer U1.23 (P0.20)
- net MIC_I2S_WS: now also U1.8 (P0.06); no longer U1.28 (P0.23)
Changed lines of the file:
@@
 Text GLabel 1500 2400 2    60   Input ~ 0
 ACC_I2C_SDA
-Text GLabel 6800 4200 2    60   Input ~ 0
+Text GLabel 6800 2000 2    60   Input ~ 0
 APA102_1_MOSI
-Text GLabel 6800 4300 2    60   Input ~ 0
+Text GLabel 6800 1900 2    60   Input ~ 0
 APA102_1_SCK
-Text GLabel 6800 4100 2    60   Input ~ 0
+Text GLabel 6800 1700 2    60   Input ~ 0
 APA102_0_SCK
-Text GLabel 6800 4000 2    60   Input ~ 0
+Text GLabel 6800 1800 2    60   Input ~ 0
 APA102_0_MOSI
+Text GLabel 6800 2200 2    60   Input ~ 0
+MIC_I2S_SCK
+Text GLabel 6800 2100 2    60   Input ~ 0
+MIC_I2S_WS
+Text GLabel 6800 2300 2    60   Input ~ 0
+MIC_I2S_SD
 Text GLabel 6800 3700 2    60   Input ~ 0
-MIC_I2S_SCK
+ACC_I2C_SCL
 Text GLabel 6800 3800 2    60   Input ~ 0
-MIC_I2S_WS
-Text GLabel 6800 3500 2    60   Input ~ 0
-MIC_I2S_SD
-Text GLabel 6800 2100 2    60   Input ~ 0
-ACC_I2C_SCL
-Text GLabel 6800 2200 2    60   Input ~ 0
 ACC_I2C_SDA
 Text GLabel 10350 1400 2    60   Input ~ 0
@@
 	6800 3700 6700 3700
 Wire Wire Line
-	6700 4000 6800 4000
-Wire Wire Line
-	6800 4100 6700 4100
-Wire Wire Line
-	6700 4200 6800 4200
-Wire Wire Line
-	6800 4300 6700 4300
+	6700 1700 6800 1700
+Wire Wire Line
+	6800 1800 6700 1800
+Wire Wire Line
+	6700 1900 6800 1900
+Wire Wire Line
+	6800 2000 6700 2000
 Wire Wire Line
 	1500 3500 1400 3500
@@
 Wire Wire Line
 	8200 2500 8100 2500
+Wire Wire Line
+	6800 2300 6700 2300
 $EndSCHEMATC
