File: hardware/power.sch (KiCad schematic (older format))
At the start: 20 parts, among them SW1 PM_BTN, U2 TPS63031DSKR, U5 BQ24075RGTT, U6 MAX16054AZT+T, U7 sip32408

Commit message: Fixed SIP32408 footprint pins/pads lacking GND
Connections:
- net GND: now also U7.2 (GND), U7.5 (GND)
Changed lines of the file:
@@
 	5150 6550 5250 6550
 Wire Wire Line
-	5250 6550 5250 6700
+	5250 6550 5250 6800
 Wire Wire Line
 	5250 6700 5150 6700
@@
 Wire Wire Line
 	1800 6750 1800 6850
+$Comp
+L GND #PWR?
+U 1 1 58AA4391
+P 5250 6800
+F 0 "#PWR?" H 5300 6850 50  0001 C CNN
+F 1 "GND" H 5255 6627 50  0000 C CNN
+F 2 "" H -250 0   50  0001 C CNN
+F 3 "" H -250 0   50  0001 C CNN
+	1    5250 6800
+	1    0    0    -1
+$EndComp
+Connection ~ 5250 6700
 $EndSCHEMATC
